File: hw/esp03-breakout.kicad_pcb (KiCad board)
At the start: 2 copper layers, 61 x 49.5 mm, 16 parts, among them P1 JTAG, P2 SERIAL, P3 CONN_2, SW1 SWITCH_INV2, SW2 SWITCH_INV2, U1 ESP8266-ESP03

Commit message: hw/esp03-breakout: shrink the board, fix bugs, update drawings
Flip connectors, jumpers and buttons to the back side.

Signed-off-by: Max Filippov <jcmvbkbc@gmail.com>
Parts:
- JP1, JP2, JP3, P1, P2, SW1, SW2: moved to B.Cu
- moved P3 208.5 mm to (240.0, 30.5), turned to 180 degrees
- moved R1 207.0 mm to (266.7, 59.7), turned to 180 degrees
- moved R2 207.0 mm to (266.7, 55.9), turned to 180 degrees
- moved R3 207.0 mm to (266.7, 52.1), turned to 180 degrees
- moved P1 205.7 mm to (243.8, 50.8), turned to 270 degrees
- moved JP1 194.3 mm to (260.4, 59.7), turned to 180 degrees
- moved JP2 194.3 mm to (260.4, 54.6), turned to 180 degrees
- moved JP3 194.3 mm to (260.4, 49.5), turned to 180 degrees
- moved U1 194.3 mm to (261.6, 36.8)
- moved C1 193.1 mm to (270.5, 40.6), turned to 270 degrees
- moved SW1 193.0 mm to (254.0, 66.0)
- moved SW2 191.8 mm to (262.9, 66.0)
- moved P2 184.2 mm to (233.7, 50.8), turned to 270 degrees
- moved R4 181.6 mm to (254.0, 59.7), turned to 180 degrees
- moved R5 181.6 mm to (254.0, 55.9), turned to 180 degrees
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Routing:
- net GND: track 184.7 -> 270.3 mm
- net VCC: track 47.2 -> 77.5 mm, vias 0 -> 1
- net /MTMS: track 40.6 -> 21.1 mm, vias 0 -> 2
- net /MTCK: track 56.2 -> 37.7 mm
- net /MTDI: track 40.8 -> 26.6 mm
- net /MTDO: track 84.2 -> 73.9 mm
- net N-0000034: track 100.9 -> 90.8 mm
- net N-000004: track 12.0 -> 20.2 mm
- net /TX: track 87.6 -> 79.9 mm, vias 0 -> 2
- net /RX: track 82.7 -> 76.9 mm, vias 0 -> 2
- net N-000003: track 20.4 -> 15.1 mm
- net N-000001: track 3.91 -> 7.50 mm
- net N-0000013: track 3.38 -> 4.97 mm
- net N-000002: track 3.38 -> 4.97 mm
- added copper zone on F.Cu, net GND
Other:
- board size 61 x 49.5 mm -> 49.5 x 49.5 mm
- net class Default: clearance 0.254 -> 0.3; trace_width 0.254 -> 0.3
- rule trace_clearance: 0.254 -> 0.3
- board text added: "ESP03-breakout v.0.2"
